File: QuantizerFront/QuantizerFront.kicad_pcb (KiCad board)
At the start: 2 copper layers, 100 x 95 mm, 61 parts, among them J16 Conn_01x07_Female, U2 74HC165, U3 74HC595, U4 74HC165, U5 74HC595

Commit message: Gerber Updates
Parts:
- J16: moved to B.Cu
- turned J16 to 180 degrees
Changed lines of the file:
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@@
-    )
-  )
-  (footprint "Connector_PinSocket_2.54mm:PinSocket_1x07_P2.54mm_Vertical" (layer "F.Cu")
-    (at 160.025 92.4)
-    (descr "Through hole straight socket strip, 1x07, 2.54mm pitch, single row (from Kicad 4.0.7), script generated")
-    (tags "Through hole socket strip THT 1x07 2.54mm single row")
-    (property "Sheetfile" "QuantizerFront.kicad_sch")
-    (property "Sheetname" "")
-    (attr through_hole)
-    (fp_text reference "J16" (at 0 -2.77) (layer "F.SilkS")
-      (effects (font (size 1 1) (thickness 0.15)))
-    )
-    (fp_text value "Conn_01x07_Female" (at 0 18.01) (layer "F.Fab")
-      (effects (font (size 1 1) (thickness 0.15)))
-    )
-    (fp_text user "${REFERENCE}" (at 0 7.62 90) (layer "F.Fab")
-      (effects (font (size 1 1) (thickness 0.15)))
-    )
-    (fp_line (start 0 -1.33) (end 1.33 -1.33) (layer "F.SilkS") (width 0.12))
-    (fp_line (start -1.33 1.27) (end -1.33 16.57) (layer "F.SilkS") (width 0.12))
-    (fp_line (start -1.33 16.57) (end 1.33 16.57) (layer "F.SilkS") (width 0.12))
-    (fp_line (start -1.33 1.27) (end 1.33 1.27) (layer "F.SilkS") (width 0.12))
-    (fp_line (start 1.33 -1.33) (end 1.33 0) (layer "F.SilkS") (width 0.12))
-    (fp_line (start 1.33 1.27) (end 1.33 16.57) (layer "F.SilkS") (width 0.12))
-    (fp_line (start 1.75 -1.8) (end 1.75 17) (layer "F.CrtYd") (width 0.05))
-    (fp_line (start -1.8 -1.8) (end 1.75 -1.8) (layer "F.CrtYd") (width 0.05))
-    (fp_line (start -1.8 17) (end -1.8 -1.8) (layer "F.CrtYd") (width 0.05))
-    (fp_line (start 1.75 17) (end -1.8 17) (layer "F.CrtYd") (width 0.05))
-    (fp_line (start 1.27 16.51) (end -1.27 16.51) (layer "F.Fab") (width 0.1))
-    (fp_line (start -1.27 -1.27) (end 0.635 -1.27) (layer "F.Fab") (width 0.1))
-    (fp_line (start -1.27 16.51) (end -1.27 -1.27) (layer "F.Fab") (width 0.1))
-    (fp_line (start 1.27 -0.635) (end 1.27 16.51) (layer "F.Fab") (width 0.1))
-    (fp_line (start 0.635 -1.27) (end 1.27 -0.635) (layer "F.Fab") (width 0.1))
-    (pad "1" thru_hole rect (at 0 0) (size 1.7 1.7) (drill 1) (layers *.Cu *.Mask)
-      (net 15 "/SDI_F") (pinfunction "Pin_1") (pintype "passive"))
-    (pad "2" thru_hole oval (at 0 2.54) (size 1.7 1.7) (drill 1) (layers *.Cu *.Mask)
-      (net 11 "/SLI_F") (pinfunction "Pin_2") (pintype "passive"))
-    (pad "3" thru_hole oval (at 0 5.08) (size 1.7 1.7) (drill 1) (layers *.Cu *.Mask)
-      (net 14 "/SDO_F") (pinfunction "Pin_3") (pintype "passive"))
-    (pad "4" thru_hole oval (at 0 7.62) (size 1.7 1.7) (drill 1) (layers *.Cu *.Mask)
-      (net 13 "/SLO_F") (pinfunction "Pin_4") (pintype "passive"))
-    (pad "5" thru_hole oval (at 0 10.16) (size 1.7 1.7) (drill 1) (layers *.Cu *.Mask)
-      (net 12 "/SCL_F") (pinfunction "Pin_5") (pintype "passive"))
-    (pad "6" thru_hole oval (at 0 12.7) (size 1.7 1.7) (drill 1) (layers *.Cu *.Mask)
-      (net 1 "GND") (pinfunction "Pin_6") (pintype "passive"))
-    (pad "7" thru_hole oval (at 0 15.24) (size 1.7 1.7) (drill 1) (layers *.Cu *.Mask)
-      (net 7 "+5V_1") (pinfunction "Pin_7") (pintype "passive"))
-    (model "${KICAD6_3DMODEL_DIR}/Connector_PinSocket_2.54mm.3dshapes/PinSocket_1x07_P2.54mm_Vertical.wrl"
-      (offset (xyz 0 0 0))
-      (scale (xyz 1 1 1))
-      (rotate (xyz 0 0 0))
     )
   )
@@
       (offset (xyz 0 0 0))
       (scale (xyz 1 1 1))
+      (rotate (xyz 0 0 0))
+    )
+  )
+  (footprint "Connector_PinSocket_2.54mm:PinSocket_1x07_P2.54mm_Vertical" (layer "B.Cu")
+    (at 160.025 92.4 180)
+    (descr "Through hole straight socket strip, 1x07, 2.54mm pitch, single row (from Kicad 4.0.7), script generated")
+    (tags "Through hole socket strip THT 1x07 2.54mm single row")
+    (property "Sheetfile" "QuantizerFront.kicad_sch")
+    (property "Sheetname" "")
+    (attr through_hole)
+    (fp_text reference "J16" (at 0 2.77) (layer "B.SilkS")
+      (effects (font (size 1 1) (thickness 0.15)) (justify mirror))
+    )
+    (fp_text value "Conn_01x07_Female" (at 0 -18.01) (layer "B.Fab")
+      (effects (font (size 1 1) (thickness 0.15)) (justify mirror))
+    )
+    (fp_text user "${REFERENCE}" (at 0 -7.62 90) (layer "B.Fab")
+      (effects (font (size 1 1) (thickness 0.15)) (justify mirror))
+    )
+    (fp_line (start 0 1.33) (end 1.33 1.33) (layer "B.SilkS") (width 0.12))
+    (fp_line (start -1.33 -1.27) (end -1.33 -16.57) (layer "B.SilkS") (width 0.12))
+    (fp_line (start -1.33 -16.57) (end 1.33 -16.57) (layer "B.SilkS") (width 0.12))
+    (fp_line (start -1.33 -1.27) (end 1.33 -1.27) (layer "B.SilkS") (width 0.12))
+    (fp_line (start 1.33 1.33) (end 1.33 0) (layer "B.SilkS") (width 0.12))
+    (fp_line (start 1.33 -1.27) (end 1.33 -16.57) (layer "B.SilkS") (width 0.12))
+    (fp_line (start 1.75 1.8) (end 1.75 -17) (layer "B.CrtYd") (width 0.05))
+    (fp_line (start -1.8 1.8) (end 1.75 1.8) (layer "B.CrtYd") (width 0.05))
+    (fp_line (start -1.8 -17) (end -1.8 1.8) (layer "B.CrtYd") (width 0.05))
+    (fp_line (start 1.75 -17) (end -1.8 -17) (layer "B.CrtYd") (width 0.05))
+    (fp_line (start 1.27 -16.51) (end -1.27 -16.51) (layer "B.Fab") (width 0.1))
+    (fp_line (start -1.27 1.27) (end 0.635 1.27) (layer "B.Fab") (width 0.1))
+    (fp_line (start -1.27 -16.51) (end -1.27 1.27) (layer "B.Fab") (width 0.1))
+    (fp_line (start 1.27 0.635) (end 1.27 -16.51) (layer "B.Fab") (width 0.1))
+    (fp_line (start 0.635 1.27) (end 1.27 0.635) (layer "B.Fab") (width 0.1))
+    (pad "1" thru_hole rect (at 0 0 180) (size 1.7 1.7) (drill 1) (layers *.Cu *.Mask)
+      (net 15 "/SDI_F") (pinfunction "Pin_1") (pintype "passive"))
+    (pad "2" thru_hole oval (at 0 -2.54 180) (size 1.7 1.7) (drill 1) (layers *.Cu *.Mask)
+      (net 11 "/SLI_F") (pinfunction "Pin_2") (pintype "passive"))
+    (pad "3" thru_hole oval (at 0 -5.08 180) (size 1.7 1.7) (drill 1) (layers *.Cu *.Mask)
+      (net 14 "/SDO_F") (pinfunction "Pin_3") (pintype "passive"))
+    (pad "4" thru_hole oval (at 0 -7.62 180) (size 1.7 1.7) (drill 1) (layers *.Cu *.Mask)
+      (net 13 "/SLO_F") (pinfunction "Pin_4") (pintype "passive"))
+    (pad "5" thru_hole oval (at 0 -10.16 180) (size 1.7 1.7) (drill 1) (layers *.Cu *.Mask)
+      (net 12 "/SCL_F") (pinfunction "Pin_5") (pintype "passive"))
+    (pad "6" thru_hole oval (at 0 -12.7 180) (size 1.7 1.7) (drill 1) (layers *.Cu *.Mask)
+      (net 1 "GND") (pinfunction "Pin_6") (pintype "passive"))
+    (pad "7" thru_hole oval (at 0 -15.24 180) (size 1.7 1.7) (drill 1) (layers *.Cu *.Mask)
+      (net 7 "+5V_1") (pinfunction "Pin_7") (pintype "passive"))
+    (model "${KICAD6_3DMODEL_DIR}/Connector_PinSocket_2.54mm.3dshapes/PinSocket_1x07_P2.54mm_Vertical.wrl"
+      (offset (xyz 0 0 0))
+      (scale (xyz 1 1 1))
