File: QuantizerBack/QuantizerBack.kicad_pcb (KiCad board)
At the start: 2 copper layers, 170 x 95 mm, 128 parts, among them J1 Conn_02x03_Odd_Even, J10 GATEB, J11 INB, J12 OUTB, J13 CVA, J14 CVB, J15 Synth_power_2x5, J17 Conn_01x07_Male, J2 Conn_01x06, J5 TRIGA, J6 GATEA, J7 INA, J8 OUTA, J9 TRIGB, Q1 2N3904, Q2 2N3904, U1 ATmega328P-P, U10 LP2951-5.0, U6 TL074, U7 TL074, U8 TL072, U9 L78L05_TO92, Y1 16MHz

Commit message: Fix Trigger Input Jack Issue
Previous version of these boards did not have the tip normal of the input jacks connected to +12v to allow free running mode. Kassutronics updated the documentation to add a resistor that prevents shorting in this connection. This update connects the tip normal in the input jacks to +12v through a 10k resistor.
Parts:
- removed J15: Synth_power_2x5, ao_tht:Power_Header
- added J3: Synth_power_2x5_passive, AO_tht:Power_Header, B.Cu at (142.9, 139.2)
- added R235: 10k, AO_tht:R_Axial_DIN0207_L6.3mm_D2.5mm_P10.16mm_Horizontal, B.Cu at (187.2, 141.7)
- added R236: 10k, AO_tht:R_Axial_DIN0207_L6.3mm_D2.5mm_P10.16mm_Horizontal, B.Cu at (203.8, 100.0)
- U10: value LP2951-5.0 -> LP2951-5.0_DIP
Connections:
- J5 pad TN: /12V -> Net-(J5-PadTN)
- J9 pad TN: /12VJ -> Net-(J9-PadTN)
Routing:
- net +12V_1: track 235.4 -> 286.8 mm
- net Net-(J5-PadTN): track 0.00 -> 11.2 mm
- net Net-(J9-PadTN): track 0.00 -> 9.52 mm
- net +5V_1: track 142.5 -> 145.0 mm
- net Net-(U1-PD7): track 42.1 -> 44.0 mm
- net Net-(J2-Pin_6): track 27.1 -> 28.5 mm
- net /INA: track 102.9 -> 104.2 mm
- net /OUTA: track 136.2 -> 137.4 mm
- net /ADC0: track 24.2 -> 24.9 mm
- net /SCL: track 22.1 -> 22.8 mm
- net GND: vias 4 -> 7
