File: QuantizerBack/QuantizerBack.kicad_sch (KiCad schematic)
At the start: 128 parts, among them J1 Conn_02x03_Odd_Even, J10 GATEB, J11 INB, J12 OUTB, J13 CVA, J14 CVB, J15 Synth_power_2x5, J17 Conn_01x07_Male, J2 Conn_01x06, J5 TRIGA, J6 GATEA, J7 INA, J8 OUTA, J9 TRIGB, Q1 2N3904, Q2 2N3904, U1 ATmega328P-P, U10 LP2951-5.0_DIP, U6 TL074, U7 TL074, U8 TL072, U9 L78L05_TO92, Y1 16MHz

Commit message: Fix Trigger Input Jack Issue
Previous version of these boards did not have the tip normal of the input jacks connected to +12v to allow free running mode. Kassutronics updated the documentation to add a resistor that prevents shorting in this connection. This update connects the tip normal in the input jacks to +12v through a 10k resistor.
Parts:
- removed J15: Synth_power_2x5, ao_tht:Power_Header, symbol ao_symbols:Synth_power_2x5
- added J3: Synth_power_2x5_passive, AO_tht:Power_Header, symbol AO_symbols:Synth_power_2x5_passive
- added R235, R236: 10k, AO_tht:R_Axial_DIN0207_L6.3mm_D2.5mm_P10.16mm_Horizontal, symbol ao_symbols:R
Connections:
- net +12V_1: now also R235.2, R236.2
- net GND: now also J3.3 (GND), J3.4 (GND), J3.5 (GND), J3.6 (GND), J3.7 (GND), J3.8 (GND)
- net at L2.2: now also J3.1 (-12V), J3.2 (-12V)
- net at L1.2: now also J3.10 (+12V), J3.9 (+12V)
- net 12V: no longer names the net of J5.TN
- net 12V: now also R235.1
- net 12VJ: no longer names the net of J9.TN
- net 12VJ: now also R236.1
Other:
- moved on the sheet: C10, C11, C16, C17, C22, C23, C24, C25, J5, J9, L1, L2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
